File: Nano-Breakout.kicad_sch (KiCad schematic)
At the start: 3 parts, among them J101 Conn_01x15, J102 Conn_01x15

Commit message: Production
Parts:
- A101, J101, J102: now left out of the parts list
Changed lines of the file:
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@@
   (junction (at 155.575 85.725) (diameter 0) (color 0 0 0 0)
   )
+  (junction (at 137.795 72.39) (diameter 0) (color 0 0 0 0)
+  )
   (junction (at 144.145 125.095) (diameter 0) (color 0 0 0 0)
   )
+  (junction (at 144.145 127) (diameter 0) (color 0 0 0 0)
+  )
   (wire (pts (xy 137.795 72.39) (xy 140.335 72.39))
     (stroke (width 0) (type default) (color 0 0 0 0))
@@
     (stroke (width 0) (type default) (color 0 0 0 0))
   )
+  (wire (pts (xy 125.73 125.73) (xy 125.73 127))
+    (stroke (width 0) (type default) (color 0 0 0 0))
+  )
   (wire (pts (xy 144.145 125.095) (xy 145.415 125.095))
     (stroke (width 0) (type default) (color 0 0 0 0))
@@
     (stroke (width 0) (type default) (color 0 0 0 0))
   )
+  (wire (pts (xy 144.145 127) (xy 144.145 127.635))
+    (stroke (width 0) (type default) (color 0 0 0 0))
+  )
   (wire (pts (xy 155.575 114.935) (xy 170.815 114.935))
     (stroke (width 0) (type default) (color 0 0 0 0))
@@
     (stroke (width 0) (type default) (color 0 0 0 0))
   )
+  (wire (pts (xy 127 69.85) (xy 127 72.39))
+    (stroke (width 0) (type default) (color 0 0 0 0))
+  )
   (wire (pts (xy 113.665 84.455) (xy 119.38 84.455))
     (stroke (width 0) (type default) (color 0 0 0 0))
@@
     (stroke (width 0) (type default) (color 0 0 0 0))
   )
+  (wire (pts (xy 125.73 127) (xy 144.145 127))
+    (stroke (width 0) (type default) (color 0 0 0 0))
+  )
   (wire (pts (xy 170.18 69.85) (xy 170.18 94.615))
     (stroke (width 0) (type default) (color 0 0 0 0))
   )
-  (wire (pts (xy 144.145 125.095) (xy 144.145 127.635))
+  (wire (pts (xy 144.145 125.095) (xy 144.145 127))
     (stroke (width 0) (type default) (color 0 0 0 0))
   )
@@
   )
   (wire (pts (xy 137.795 69.85) (xy 137.795 72.39))
+    (stroke (width 0) (type default) (color 0 0 0 0))
+  )
+  (wire (pts (xy 127 72.39) (xy 137.795 72.39))
     (stroke (width 0) (type default) (color 0 0 0 0))
   )
@@
   )
   (symbol (lib_id "MCU_Module:Arduino_Nano_v3.x") (at 142.875 99.695 0) (unit 1)
-    (in_bom yes) (on_board yes) (fields_autoplaced)
+    (in_bom no) (on_board yes) (fields_autoplaced)
     (property "Reference" "A101" (id 0) (at 147.4344 125.73 0)
       (effects (font (size 1.27 1.27)) (justify left))
@@
     (pin "1")
   )
+  (symbol (lib_id "power:PWR_FLAG") (at 127 69.85 0) (unit 1)
+    (in_bom yes) (on_board yes) (fields_autoplaced)
+    (property "Reference" "#FLG0101" (id 0) (at 127 67.945 0)
+      (effects (font (size 1.27 1.27)) hide)
+    )
+    (property "Value" "PWR_FLAG" (id 1) (at 127 64.77 0))
+    (property "Footprint" "" (id 2) (at 127 69.85 0)
+      (effects (font (size 1.27 1.27)) hide)
+    )
+    (property "Datasheet" "~" (id 3) (at 127 69.85 0)
+      (effects (font (size 1.27 1.27)) hide)
+    )
+    (pin "1")
+  )
   (symbol (lib_id "Connector_Generic:Conn_01x15") (at 108.585 97.155 0) (mirror y) (unit 1)
-    (in_bom yes) (on_board yes) (fields_autoplaced)
+    (in_bom no) (on_board yes) (fields_autoplaced)
     (property "Reference" "J101" (id 0) (at 108.585 72.39 0))
     (property "Value" "Conn_01x15" (id 1) (at 108.585 74.93 0))
@@
     (pin "9")
   )
+  (symbol (lib_id "power:PWR_FLAG") (at 125.73 125.73 0) (mirror y) (unit 1)
+    (in_bom yes) (on_board yes) (fields_autoplaced)
+    (property "Reference" "#FLG0102" (id 0) (at 125.73 123.825 0)
+      (effects (font (size 1.27 1.27)) hide)
+    )
+    (property "Value" "PWR_FLAG" (id 1) (at 125.73 120.65 0))
+    (property "Footprint" "" (id 2) (at 125.73 125.73 0)
+      (effects (font (size 1.27 1.27)) hide)
+    )
+    (property "Datasheet" "~" (id 3) (at 125.73 125.73 0)
+      (effects (font (size 1.27 1.27)) hide)
+    )
+    (pin "1")
+  )
   (symbol (lib_id "power:GND") (at 144.145 127.635 0) (unit 1)
     (in_bom yes) (on_board yes) (fields_autoplaced)
@@
   )
   (symbol (lib_id "Connector_Generic:Conn_01x15") (at 175.895 109.855 0) (unit 1)
-    (in_bom yes) (on_board yes) (fields_autoplaced)
+    (in_bom no) (on_board yes) (fields_autoplaced)
     (property "Reference" "J102" (id 0) (at 179.07 108.5849 0)
       (effects (font (size 1.27 1.27)) (justify left))
@@
   )
   (symbol_instances
+    (path "/7954b01e-da18-4b88-8ac2-e5b2a8846eef"
+      (reference "#FLG0101") (unit 1) (value "PWR_FLAG") (footprint "")
+    )
+    (path "/a5f51278-4b8f-45e5-9a33-3b0953ea5b62"
+      (reference "#FLG0102") (unit 1) (value "PWR_FLAG") (footprint "")
+    )
     (path "/b6ea14bb-7704-4805-b88e-411989e1e0c4"
       (reference "#PWR0101") (unit 1) (value "GND") (footprint "")

Commit message: Added 3D stacking header
Parts:
- A101: footprint Module:Arduino_Nano -> Nano:Arduino_Nano
Changed lines of the file:
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@@
       (effects (font (size 1.27 1.27)) (justify left))
     )
-    (property "Footprint" "Module:Arduino_Nano" (id 2) (at 142.875 99.695 0)
+    (property "Footprint" "Nano:Arduino_Nano" (id 2) (at 142.875 99.695 0)
       (effects (font (size 1.27 1.27) italic) hide)
     )
@@
     )
     (path "/3955bb7e-0cab-4a30-88b1-ae5ad69932b2"
-      (reference "A101") (unit 1) (value "Arduino_Nano_v3.x") (footprint "Module:Arduino_Nano")
+      (reference "A101") (unit 1) (value "Arduino_Nano_v3.x") (footprint "Nano:Arduino_Nano")
     )
     (path "/8390c402-6605-414b-b5f9-3b111ad0c236"

Commit message: Names streamlined
Parts:
- A101: footprint Nano:Arduino_Nano -> Nano:Arduino_Nano_Stacking_THT
Changed lines of the file:
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@@
       (effects (font (size 1.27 1.27)) (justify left))
     )
-    (property "Footprint" "Nano:Arduino_Nano" (id 2) (at 142.875 99.695 0)
+    (property "Footprint" "Nano:Arduino_Nano_Stacking_THT" (id 2) (at 142.875 99.695 0)
       (effects (font (size 1.27 1.27) italic) hide)
     )
@@
     )
     (path "/3955bb7e-0cab-4a30-88b1-ae5ad69932b2"
-      (reference "A101") (unit 1) (value "Arduino_Nano_v3.x") (footprint "Nano:Arduino_Nano")
+      (reference "A101") (unit 1) (value "Arduino_Nano_v3.x") (footprint "Nano:Arduino_Nano_Stacking_THT")
     )
     (path "/8390c402-6605-414b-b5f9-3b111ad0c236"
